File: Schematics/Sensor/GaussMouse_Sensor.kicad_pcb (KiCad board)
At the start: 2 copper layers, 46 x 46 mm, 47 parts, among them J1 Prog, J2 Conn_01x02, J3 OledDisplay, J4 Conn_01x09, SW1 SW_Push_45deg, SW2 SW_Push_45deg, SW3 SW_Push_45deg, U1 BNO085, U2 CH32V003F4P6, Y1 Crystal_Small

Commit message: Commit for backup. Short on sensor board so I'm going to redo it
Parts:
- removed J3: OledDisplay, Connector_PinHeader_2.54mm:PinHeader_1x04_P2.54mm_Vertical
- removed JP1: JOpen, Jumper:SolderJumper-2_P1.3mm_Open_TrianglePad1.0x1.5mm
- removed JP2: JClosed, Jumper:SolderJumper-2_P1.3mm_Bridged_Pad1.0x1.5mm
- removed JP3: Jumper_2_Open, Jumper:SolderJumper-2_P1.3mm_Open_TrianglePad1.0x1.5mm
- removed JP4: Jumper_2_Bridged, Jumper:SolderJumper-2_P1.3mm_Bridged_Pad1.0x1.5mm
- moved D4 43.1 mm to (138.1, 72.5), turned to 180 degrees
- moved D8 42.9 mm to (137.8, 115.4), turned to 0 degrees
- moved D5 42.8 mm to (122.8, 78.9), turned to -135 degrees
- moved D7 42.6 mm to (123.1, 109.2), turned to -45 degrees
- moved D3 42.5 mm to (153.0, 78.9), turned to 135 degrees
- moved D1 42.4 mm to (152.5, 109.4), turned to 45 degrees
- moved D2 42.0 mm to (159.0, 93.7), turned to 90 degrees
- moved D6 42.0 mm to (117.0, 93.9), turned to -90 degrees
- moved JP6 24.0 mm to (142.0, 76.5), turned to 90 degrees
- moved JP5 20.8 mm to (145.5, 76.5), turned to 90 degrees
- moved RN1 18.3 mm to (146.1, 92.3), turned to 0 degrees
- moved C6 0.45 mm to (142.0, 89.0)
- turned C4 to 180 degrees
- turned C5 to 180 degrees
- turned JP7 to 0 degrees
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- renumbered D4 to D1, D5 to D2, D6 to D3, D7 to D4, D8 to D5, D1 to D6, D2 to D7, D3 to D8
Connections:
- net PC6 renamed WS2812
- RN1 pad 3: Env_SCL -> Env_SDA
- RN1 pad 4: Env_SDA -> Env_SCL
- SW1 pad 1: PD5 -> Center
- SW2 pad 1: PD6 -> Right
- SW3 pad 1: PD7 -> Left
- U2 pad 17: unconnected-(U2-PC7-Pad17) -> Right
- U2 pad 19: unconnected-(U2-PD2-Pad19) -> Center
- U2 pad 20: unconnected-(U2-PD3-Pad20) -> Left
- U2 pad 4: PD7 -> IntN
- U2 pad 6: IntN -> unconnected-(U2-PA2-Pad6)
Routing:
- net VCC: track 0.00 -> 192.4 mm, vias 0 -> 6
- net SDA: track 0.00 -> 50.0 mm, vias 0 -> 1
- net SCL: track 0.00 -> 49.3 mm, vias 0 -> 1
- net SWIO: track 0.00 -> 45.7 mm, vias 0 -> 1
- net Center: track 0.00 -> 41.0 mm, vias 0 -> 1
- net Right: track 0.00 -> 35.4 mm, vias 0 -> 1
- net Left: track 0.00 -> 35.1 mm, vias 0 -> 1
- net VSS: track 0.00 -> 26.0 mm, vias 0 -> 47
- net CLK: track 0.00 -> 23.3 mm, vias 0 -> 1
- net MISO: track 0.00 -> 21.5 mm, vias 0 -> 1
- net PS1: track 0.00 -> 19.5 mm, vias 0 -> 3
- net Net-(D5-DOUT): track 0.00 -> 16.9 mm
- net CS: track 0.00 -> 16.7 mm, vias 0 -> 2
- net Net-(D1-DOUT): track 0.00 -> 16.1 mm
- net Net-(D4-DOUT): track 0.00 -> 16.0 mm
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- added copper zone on B.Cu, net VSS
- added copper zone on F.Cu, net VSS
